Commit message: DepthMam

File: my_gazebo/description/example_gazebo.xacro (robot description, xacro)
@@ -25,4 +25,5 @@
         </plugin>
     </gazebo>
+    <!--ros2 topic pub -1 /set_joint_trajectory trajectory_msgs/msg/JointTrajectory  '{header: {frame_id: world}, joint_names: [RL-1-1, LL-1-1], points: [  {positions: {0.8,0.6}} ]}' -->
     <gazebo>
         <plugin name="gazebo_ros_joint_pose_trajectory"
@@ -31,3 +32,42 @@
         </plugin>
     </gazebo>
+    <joint name="camera_optical_joint" type="fixed">
+        <origin xyz="0 0 0" rpy="-1.571 0 -1.571" />
+        <parent link="camera_link" />
+        <child link="camera_link_optical" />
+    </joint>
+    <link name="camera_link_optical"></link>
+    <!-- Add a gazebo tag for the ORIGINAL camera_link (but in the plugin we reference the optical frame so that ROS can orient things correctly) -->
+    <!-- Within the gazebo tag we have the sensor tag, and inside that there is (among other things) the camera tag with the camera parameters,
+            and the plugin tag with some extra parameters the plugin needs. -->
+    <!-- Note that although visualise is set to true, it won't actually visualise the depth camera in gazebo. To see the preview,
+            try swapping "depth" to "camera"-->
+    <gazebo reference="camera_link">
+        <sensor type="depth" name="Camera">
+            <update_rate>20</update_rate>
+            <visualize>true</visualize>
+            <camera name="cam">
+                <horizontal_fov>1.3962634</horizontal_fov>
+                <image>
+                    <width>640</width>
+                    <height>480</height>
+                    <format>R8B8G8</format>
+                </image>
+                <clip>
+                    <near>0.02</near>
+                    <far>300</far>
+                </clip>
+                <noise>
+                    <type>gaussian</type>
+                    <mean>0.0</mean>
+                    <stddev>0.007</stddev>
+                </noise>
+            </camera>
+            <plugin name="camera_controller" filename="libgazebo_ros_camera.so">
+                <frame_name>camera_link_optical</frame_name>
+                <min_depth>0.1</min_depth>
+                <max_depth>500</max_depth>
+            </plugin>
+        </sensor>
+    </gazebo>
 </robot>

File: my_gazebo/description/example_robot.urdf.xacro (robot description, xacro)
@@ -14,14 +14,12 @@
     <xacro:property name="base_path" value="file:////home/zega/Desktop/ros_dev/src/my_gazebo/meshes/base.dae" />
     <xacro:property name="arm_path" value="file:////home/zega/Desktop/ros_dev/src/my_gazebo/meshes/leg-section.dae" />
-    <!--
+    <!---->
 	<link name="world"></link>
--->
-    <!--BODY
+    <!--BODY-->
 	<joint name="base" type="fixed">
-		<origin xyz="2.0 2.0 0.2" />
+		<origin xyz="0 0 0.3 " />
 		<parent link="world" />
 		<child link="base_link" />
 	</joint>
-    -->
 	<link name="base_link">
 		<visual>

Commit message: lidar

File: my_gazebo/description/example_gazebo.xacro (robot description, xacro)
@@ -71,3 +71,39 @@
         </sensor>
     </gazebo>
+    <gazebo reference="RL-1-3_link">
+        <mu1 value="10.0"/> <!-- Коэффициент статического трения -->
+        <mu2 value="10.0"/> <!-- Коэффициент динамического трения -->
+        <kp value="1000000.0"/> <!-- Коэффициент жесткости контакта -->
+        <kd value="1.0"/> <!-- Коэффициент демпфирования контакта -->
+   </gazebo>
+    <gazebo reference="RL-2-3_link">
+        <mu1 value="10.0"/> <!-- Коэффициент статического трения -->
+        <mu2 value="10.0"/> <!-- Коэффициент динамического трения -->
+        <kp value="1000000.0"/> <!-- Коэффициент жесткости контакта -->
+        <kd value="1.0"/> <!-- Коэффициент демпфирования контакта -->
+    </gazebo>
+    <gazebo reference="RL-3-3_link">
+        <mu1 value="10.0"/> <!-- Коэффициент статического трения -->
+        <mu2 value="10.0"/> <!-- Коэффициент динамического трения -->
+        <kp value="1000000.0"/> <!-- Коэффициент жесткости контакта -->
+        <kd value="1.0"/> <!-- Коэффициент демпфирования контакта -->
+    </gazebo>
+    <gazebo reference="LL-1-3_link">
+        <mu1 value="10"/>
+        <mu2 value="10"/>
+        <kp value="1000000.0"/>
+        <kd value="1.0"/>
+    </gazebo>
+    <gazebo reference="LL-2-3_link">
+        <mu1 value="10"/>
+        <mu2 value="10"/>
+        <kp value="1000000.0"/>
+        <kd value="1.0"/>
+    </gazebo>
+    <gazebo reference="LL-3-3_link">
+        <mu1 value="10"/>
+        <mu2 value="10"/>
+        <kp value="1000000.0"/>
+        <kd value="1.0"/>
+    </gazebo>
 </robot>

File: my_gazebo/description/example_robot.urdf.xacro (robot description, xacro)
@@ -1,20 +1,8 @@
 <?xml version="1.0"?>
 <robot xmlns:xacro="http://www.ros.org/wiki/xacro"  name="INSECTOIDv1">
-    <!--Phys macro-->
-	<xacro:macro name="inertial_box" params="mass x y z *origin">
-		<inertial>
-			<xacro:insert_block name="origin"/>
-			<mass value="${mass}" />
-			<inertia ixx="${(1/12) * mass * (y*y+z*z)}" ixy="0.0" ixz="0.0"
-                    iyy="${(1/12) * mass * (x*x+z*z)}" iyz="0.0"
-                    izz="${(1/12) * mass * (x*x+y*y)}" />
-		</inertial>
-	</xacro:macro>
-<!--Models-->
-    <xacro:property name="base_path" value="file:////home/zega/Desktop/ros_dev/src/my_gazebo/meshes/base1.dae" />
-    <xacro:property name="arm_path_1" value="file:////home/zega/Desktop/ros_dev/src/my_gazebo/meshes/l-1.dae" />
-    <xacro:property name="arm_path_2" value="file:////home/zega/Desktop/ros_dev/src/my_gazebo/meshes/l-2.dae" />
-    <xacro:property name="arm_path_3" value="file:////home/zega/Desktop/ros_dev/src/my_gazebo/meshes/l-3.dae" />
-    <xacro:property name="camera" value="file:////home/zega/Desktop/ros_dev/src/my_gazebo/meshes/kinect.dae" />
+    <xacro:include filename="patterns.xacro"/>
+    <xacro:include filename="example_gazebo.xacro" />
+    <xacro:include filename="ros2_control.xacro"/>
+    <xacro:include filename="lidar.xacro"/>
     <!--
 	<link name="world"></link>
@@ -37,10 +25,4 @@
 			</material>
 		</visual>
-		<collision>
-			<origin xyz="0 0 0" rpy="0 0 0"/>
-			<geometry>
-				<box size="0.2 0.45 0.06" />
-			</geometry>
-		</collision>
 		<xacro:inertial_box mass="0.1" x="0.2" y="0.45" z="0.06">
             <origin xyz="0.0 0 0" rpy="0 0 0"/>
@@ -54,11 +36,5 @@
         <child link="camera_link"/>
     </joint>
-    <material name="black">
-        <color rgba="0 0 0 1"/>
-    </material>
-    <!-- camera_link describes the camera at the end of the arm -->
-    <!-- - It has multiple visual elements, which ultimately get combined together -->
-    <!-- - Even if we specify different materials, RViz will just colour them all the same as the first -->
-    <!-- - Although we could also specify multiple collision geometries, instead we just use a single box that encompasses the whole camera -->
+    <!-- camera_link describes the camera -->
     <link name="camera_link">
         <visual>
@@ -67,5 +43,4 @@
 				<mesh filename="${camera}"/>
 			</geometry>
-            <material name="black" />
         </visual>
         <visual>
@@ -76,77 +51,12 @@
             <material name="black" />
         </visual>
-        <collision>
-            <origin xyz="0.0 0 0" rpy="0 0 0"/>
-            <geometry>
-                <box size="0.12 0.15 0.15" />
-            </geometry>
-        </collision>
-        <xacro:inertial_box mass="0.1" x="0.12" y="0.15" z="0.15">
+        <xacro:inertial_box mass="0.1" x="0.12" y="0.06" z="0.12">
             <origin xyz="0.0 0 0" rpy="0 0 0"/>
         </xacro:inertial_box>
     </link>
     <!---->
-    <material name="orange">
-		<color rgba="1 0.3 0.1 1"/>
-	</material>
-    <!--LEG MACROS-->
-    <xacro:macro name="leg_section_joint" params="joint_name joint_axis joint_xyz joint_parent joint_child lower_limit upper_limit ">
-		<joint name="${joint_name}" type="revolute">
-		    <origin xyz="${joint_xyz}" />
-		    <parent link="${joint_parent}" />
-		    <child link="${joint_child}" />
-		    <axis xyz="${joint_axis}"/>
-		    <limit lower="${lower_limit}" upper="${upper_limit}" velocity="100" effort="100"/>
-            <dynamics damping="1.2" friction="1.2"/>
-	    </joint>
-    </xacro:macro>
-    <xacro:macro name="leg_section_link" params="link_name link_xyz link_rpy model">
-        <link name="${link_name}">
-		    <visual>
-			    <origin xyz="${link_xyz}" rpy="${link_rpy}"/>
-			    <geometry>
-			    	<mesh filename="${model}"/>
-			    </geometry>
-			    <material name="orange" />
-		    </visual>
-		    <collision>
-			    <origin xyz="${link_xyz}" rpy="${link_rpy}"/>
-			    <geometry>
-				    <mesh filename="${model}"/>
-			    </geometry>
-		    </collision>
-		    <xacro:inertial_box mass="0.5" x="0.09" y="0.02" z="0.2">
-			    <origin xyz="${link_xyz}" rpy="${link_rpy}"/>
-		    </xacro:inertial_box>
-	    </link>
-	</xacro:macro>
     <!---->
-    <!--LEFT 1-nd-->
-	<joint name="LL-1-1" type="revolute">
-		<origin xyz="0.07 -0.154663 0.06" />
-		<parent link="base_link" />
-		<child link="LL-1-1_link" />
-		<axis xyz="0 0 1"/>
-		<limit lower="${-(pi/4)}" upper="${pi/4}" velocity="100" effort="100"/>
-        <dynamics damping="1.2" friction="1.2"/>
-	</joint>
-	<link name="LL-1-1_link">
-		<visual>
-			<origin xyz="0.04 0 -0.04" rpy="0 ${-(pi/2)} 0"/>
-			<geometry>
-				<mesh filename="${arm_path_1}"/>
-			</geometry>
-			<material name="orange" />
-		</visual>
-		<collision>
-			<origin xyz="0.04 0 -0.04" rpy="0 ${-(pi/2)} 0"/>
-			<geometry>
-				<mesh filename="${arm_path_1}"/>
-			</geometry>
-		</collision>
-		<xacro:inertial_box mass="0.5" x="0.03" y="0.015" z="0.1">
-			<origin xyz="0.04 0 -0.04" rpy="0 ${-(pi/2)} 0"/>
-		</xacro:inertial_box>
-	</link>
+    <xacro:leg_section_joint joint_name="LL-1-1" joint_axis="0 0 1" joint_xyz="0.07 -0.154663 0.06" joint_parent="base_link" joint_child="LL-1-1_link" lower_limit="${-(pi/4)}" upper_limit="${pi/4}"  />
+    <xacro:leg_section_link link_name="LL-1-1_link" link_xyz="0.04 0 -0.04" link_rpy="0 ${-(pi/2)} 0" model="${arm_path_1}" />
     <xacro:leg_section_joint joint_name="LL-1-2" joint_axis="0 1 0" joint_xyz="0.09 0 -0.04" joint_parent="LL-1-1_link" joint_child="LL-1-2_link" lower_limit="${-pi}" upper_limit="0"  />
     <xacro:leg_section_link link_name="LL-1-2_link" link_xyz="0.02 0 -0.04" link_rpy="${-(pi/6)} 0 ${(pi/2)}" model="${arm_path_2}" />
@@ -188,5 +98,3 @@
     <xacro:leg_section_joint joint_name="RL-3-3" joint_axis="0 1 0" joint_xyz="-0.04 0 -0.08" joint_parent="RL-3-2_link" joint_child="RL-3-3_link" lower_limit="-1.51" upper_limit="${pi/2}" />
     <xacro:leg_section_link link_name="RL-3-3_link" link_xyz="0 0 -0.06" link_rpy="0 0 ${pi/2}" model="${arm_path_3}"/>
-    <xacro:include filename="example_gazebo.xacro" />
-    <xacro:include filename="ros2_control.xacro"/>
 </robot>

Commit message: map not working

File: my_gazebo/description/example_gazebo.xacro (robot description, xacro)
@@ -1,35 +1,4 @@
 <?xml version="1.0"?>
 <robot xmlns:xacro="http://www.ros.org/wiki/xacro">
-    <gazebo>
-        <plugin name="gazebo_ros_joint_state_publisher"
-            filename="libgazebo_ros_joint_state_publisher.so">
-            <update_rate>20</update_rate>
-            <joint_name>RL-1-1</joint_name>
-            <joint_name>RL-1-2</joint_name>
-            <joint_name>RL-1-3</joint_name>
-            <joint_name>RL-2-1</joint_name>
-            <joint_name>RL-2-2</joint_name>
-            <joint_name>RL-2-3</joint_name>
-            <joint_name>RL-3-1</joint_name>
-            <joint_name>RL-3-2</joint_name>
-            <joint_name>RL-3-3</joint_name>
-            <joint_name>LL-1-1</joint_name>
-            <joint_name>LL-1-2</joint_name>
-            <joint_name>LL-1-3</joint_name>
-            <joint_name>LL-2-1</joint_name>
-            <joint_name>LL-2-2</joint_name>
-            <joint_name>LL-2-3</joint_name>
-            <joint_name>LL-3-1</joint_name>
-            <joint_name>LL-3-2</joint_name>
-            <joint_name>LL-3-3</joint_name>
-        </plugin>
-    </gazebo>
-    <!--ros2 topic pub -1 /set_joint_trajectory trajectory_msgs/msg/JointTrajectory  '{header: {frame_id: world}, joint_names: [RL-1-1, LL-1-1], points: [  {positions: {0.8,0.6}} ]}' -->
-    <gazebo>
-        <plugin name="gazebo_ros_joint_pose_trajectory"
-            filename="libgazebo_ros_joint_pose_trajectory.so">
-            <update_rate>20</update_rate>
-        </plugin>
-    </gazebo>
     <joint name="camera_optical_joint" type="fixed">
         <origin xyz="0 0 0" rpy="-1.571 0 -1.571" />

File: my_gazebo/description/example_robot.urdf.xacro (robot description, xacro)
@@ -5,15 +5,20 @@
     <xacro:include filename="ros2_control.xacro"/>
     <xacro:include filename="lidar.xacro"/>
-    <!--
-	<link name="world"></link>
-    -->
-    <!--BODY
-	<joint name="base" type="fixed">
-		<origin xyz="0 0 0.3 " />
-		<parent link="world" />
-		<child link="base_link" />
+    <!---->
+	<link name="base_link"></link>
+    <!--BODY -->
+     <joint name="base_footprint_joint" type="fixed">
+        <parent link="base_link"/>
+        <child link="base_footprint"/>
+        <origin xyz="0 0 0" rpy="0 0 0"/>
+    </joint>
+	<joint name="base_joint" type="fixed">
+		<origin xyz="0 0 0.01 " />
+		<parent link="base_link" />
+		<child link="robot_link" />
 	</joint>
-    -->
-	<link name="base_link">
+    <link name="base_footprint">
+    </link>
+	<link name="robot_link">
 		<visual>
 			<origin xyz="0 0 0" rpy="0 0 ${pi/2}"/>
@@ -25,5 +30,5 @@
 			</material>
 		</visual>
-		<xacro:inertial_box mass="0.1" x="0.2" y="0.45" z="0.06">
+		<xacro:inertial_box mass="3.0" x="0.2" y="0.45" z="0.06">
             <origin xyz="0.0 0 0" rpy="0 0 0"/>
         </xacro:inertial_box>
@@ -33,5 +38,5 @@
     <joint name="camera_joint" type="fixed">
         <origin xyz="0 -0.2 0.1" rpy="0 0 ${-pi/2}"/>
-        <parent link="base_link"/>
+        <parent link="robot_link"/>
         <child link="camera_link"/>
     </joint>
@@ -57,5 +62,5 @@
     <!---->
     <!---->
-    <xacro:leg_section_joint joint_name="LL-1-1" joint_axis="0 0 1" joint_xyz="0.07 -0.154663 0.06" joint_parent="base_link" joint_child="LL-1-1_link" lower_limit="${-(pi/4)}" upper_limit="${pi/4}"  />
+    <xacro:leg_section_joint joint_name="LL-1-1" joint_axis="0 0 1" joint_xyz="0.07 -0.154663 0.06" joint_parent="robot_link" joint_child="LL-1-1_link" lower_limit="${-(pi/4)}" upper_limit="${pi/4}"  />
     <xacro:leg_section_link link_name="LL-1-1_link" link_xyz="0.04 0 -0.04" link_rpy="0 ${-(pi/2)} 0" model="${arm_path_1}" />
     <xacro:leg_section_joint joint_name="LL-1-2" joint_axis="0 1 0" joint_xyz="0.09 0 -0.04" joint_parent="LL-1-1_link" joint_child="LL-1-2_link" lower_limit="${-pi}" upper_limit="0"  />
@@ -64,5 +69,5 @@
     <xacro:leg_section_link link_name="LL-1-3_link" link_xyz="0 0 -0.06" link_rpy="0 0 ${-pi/2}" model="${arm_path_3}"/>
     <!--LEFT 2-nd-->
-    <xacro:leg_section_joint joint_name="LL-2-1" joint_axis="0 0 1" joint_xyz="0.07 -0.01 0.06" joint_parent="base_link" joint_child="LL-2-1_link" lower_limit="${-pi/4}" upper_limit="${pi/4}" />
+    <xacro:leg_section_joint joint_name="LL-2-1" joint_axis="0 0 1" joint_xyz="0.07 -0.01 0.06" joint_parent="robot_link" joint_child="LL-2-1_link" lower_limit="${-pi/4}" upper_limit="${pi/4}" />
     <xacro:leg_section_link link_name="LL-2-1_link" link_xyz="0.04 0 -0.04" link_rpy="0 ${-(pi/2)} 0" model="${arm_path_1}" />
     <xacro:leg_section_joint joint_name="LL-2-2" joint_axis="0 1 0" joint_xyz="0.09 0 -0.04" joint_parent="LL-2-1_link" joint_child="LL-2-2_link" lower_limit="${-pi}" upper_limit="0" />
@@ -71,5 +76,5 @@
     <xacro:leg_section_link link_name="LL-2-3_link" link_xyz="0 0 -0.06" link_rpy="0 0 ${-pi/2}" model="${arm_path_3}"/>
 <!--LEFT 3-nd-->
-    <xacro:leg_section_joint joint_name="LL-3-1" joint_axis="0 0 1" joint_xyz="0.07 0.158646 0.06" joint_parent="base_link" joint_child="LL-3-1_link" lower_limit="${-pi/4}" upper_limit="${pi/4}" />
+    <xacro:leg_section_joint joint_name="LL-3-1" joint_axis="0 0 1" joint_xyz="0.07 0.158646 0.06" joint_parent="robot_link" joint_child="LL-3-1_link" lower_limit="${-pi/4}" upper_limit="${pi/4}" />
     <xacro:leg_section_link link_name="LL-3-1_link" link_xyz="0.04 0 -0.04" link_rpy="0 ${-(pi/2)} 0" model="${arm_path_1}"/>
     <xacro:leg_section_joint joint_name="LL-3-2" joint_axis="0 1 0" joint_xyz="0.09 0 -0.04" joint_parent="LL-3-1_link" joint_child="LL-3-2_link" lower_limit="${-pi}" upper_limit="0" />
@@ -78,5 +83,5 @@
     <xacro:leg_section_link link_name="LL-3-3_link" link_xyz="0 0 -0.06" link_rpy="0 0 ${-pi/2}" model="${arm_path_3}"/>
 <!--RIGHT 1-nd-->
-    <xacro:leg_section_joint joint_name="RL-1-1" joint_axis="0 0 1" joint_xyz="-0.07 -0.158646 0.06" joint_parent="base_link" joint_child="RL-1-1_link" lower_limit="${-pi/4}" upper_limit="${pi/4}" />
+    <xacro:leg_section_joint joint_name="RL-1-1" joint_axis="0 0 1" joint_xyz="-0.07 -0.158646 0.06" joint_parent="robot_link" joint_child="RL-1-1_link" lower_limit="${-pi/4}" upper_limit="${pi/4}" />
     <xacro:leg_section_link link_name="RL-1-1_link" link_xyz="-0.04 0 -0.04" link_rpy="0 ${(pi/2)} 0" model="${arm_path_1}"/>
     <xacro:leg_section_joint joint_name="RL-1-2" joint_axis="0 1 0" joint_xyz="-0.08 0 -0.04" joint_parent="RL-1-1_link" joint_child="RL-1-2_link" lower_limit="0" upper_limit="${pi}" />
@@ -85,5 +90,5 @@
     <xacro:leg_section_link link_name="RL-1-3_link" link_xyz="0 0 -0.06" link_rpy="0 0 ${pi/2}" model="${arm_path_3}"/>
 <!--RIGHT 2-nd-->
-    <xacro:leg_section_joint joint_name="RL-2-1" joint_axis="0 0 1" joint_xyz="-0.07 -0.01 0.06" joint_parent="base_link" joint_child="RL-2-1_link" lower_limit="${-pi/4}" upper_limit="${pi/4}" />
+    <xacro:leg_section_joint joint_name="RL-2-1" joint_axis="0 0 1" joint_xyz="-0.07 -0.01 0.06" joint_parent="robot_link" joint_child="RL-2-1_link" lower_limit="${-pi/4}" upper_limit="${pi/4}" />
     <xacro:leg_section_link link_name="RL-2-1_link" link_xyz="-0.04 0 -0.04" link_rpy="0 ${(pi/2)} 0" model="${arm_path_1}"/>
     <xacro:leg_section_joint joint_name="RL-2-2" joint_axis="0 1 0" joint_xyz="-0.08 0 -0.04" joint_parent="RL-2-1_link" joint_child="RL-2-2_link" lower_limit="0" upper_limit="${pi}" />
@@ -92,5 +97,5 @@
     <xacro:leg_section_link link_name="RL-2-3_link" link_xyz="0 0 -0.06" link_rpy="0 0 ${pi/2}" model="${arm_path_3}"/>
 <!--RIGHT 3-nd-->
-    <xacro:leg_section_joint joint_name="RL-3-1" joint_axis="0 0 1" joint_xyz="-0.07 0.158646 0.06" joint_parent="base_link" joint_child="RL-3-1_link" lower_limit="${-pi/4}" upper_limit="${pi/4}" />
+    <xacro:leg_section_joint joint_name="RL-3-1" joint_axis="0 0 1" joint_xyz="-0.07 0.158646 0.06" joint_parent="robot_link" joint_child="RL-3-1_link" lower_limit="${-pi/4}" upper_limit="${pi/4}" />
     <xacro:leg_section_link link_name="RL-3-1_link" link_xyz="-0.04 0 -0.04" link_rpy="0 ${(pi/2)} 0" model="${arm_path_1}"/>
     <xacro:leg_section_joint joint_name="RL-3-2" joint_axis="0 1 0" joint_xyz="-0.08 0 -0.04" joint_parent="RL-3-1_link" joint_child="RL-3-2_link" lower_limit="0" upper_limit="${pi}" />

File: my_gazebo/description/lidar.xacro (robot description, xacro)
@@ -1,6 +1,6 @@
 <?xml version="1.0"?>
 <robot xmlns:xacro="http://www.ros.org/wiki/xacro">
-     <joint name="laser" type="fixed">
-        <parent link="base_link"/>
+    <joint name="laser" type="fixed">
+        <parent link="robot_link"/>
         <child link="laser_frame"/>
         <origin xyz="0 0 0.06" rpy="0 0 0"/>
@@ -26,5 +26,5 @@
         <sensor name="laser" type="ray">
             <pose> 0 0 0 0 0 0 </pose>
-            <visualize>true</visualize>
+            <visualize>false</visualize>
             <update_rate>10</update_rate>
             <ray>

File: my_gazebo/description/patterns.xacro (robot description, xacro)
@@ -49,5 +49,5 @@
 		    <child link="${joint_child}" />
 		    <axis xyz="${joint_axis}"/>
-		    <limit lower="${lower_limit}" upper="${upper_limit}"  velocity="5.236" effort="0.92"/>
+		    <limit lower="${lower_limit}" upper="${upper_limit}"  velocity="50" effort="5"/>
             <dynamics damping="1.7" friction="1.7"/>
 	    </joint>

Commit message: semi-working-odom

File: my_gazebo/description/example_gazebo.xacro (robot description, xacro)
@@ -71,3 +71,29 @@
         <kd value="1.0"/>
     </gazebo>
+    <link name="imu_link"></link>
+     <joint name="imu_link_joint" type="fixed">
+        <parent link="base_link"/>
+        <child link="imu_link"/>
+        <origin xyz="0 0 0" rpy="0 0 0"/>
+    </joint>
+    <gazebo reference="imu_link">
+    <gravity>false</gravity>
+    <sensor name="imu_sensor" type="imu">
+      <always_on>true</always_on>
+      <update_rate>100</update_rate>
+      <visualize>true</visualize>
+      <topic>__default_topic__</topic>
+      <plugin filename="libgazebo_ros_imu_sensor.so" name="imu_plugin">
+        <topicName>imu</topicName>
+        <bodyName>imu_link</bodyName>
+        <updateRateHZ>10.0</updateRateHZ>
+        <gaussianNoise>0.0</gaussianNoise>
+        <xyzOffset>0 0 0</xyzOffset>
+        <rpyOffset>0 0 0</rpyOffset>
+        <frameName>imu_link</frameName>
+        <initialOrientationAsReference>false</initialOrientationAsReference>
+      </plugin>
+      <pose>0 0 0 0 0 0</pose>
+    </sensor>
+  </gazebo>
 </robot>

Commit message: GLOBAL ROBOT MOVEMENT

File: my_gazebo/description/example_gazebo.xacro (robot description, xacro)
@@ -71,29 +71,3 @@
         <kd value="1.0"/>
     </gazebo>
-    <link name="imu_link"></link>
-     <joint name="imu_link_joint" type="fixed">
-        <parent link="base_link"/>
-        <child link="imu_link"/>
-        <origin xyz="0 0 0" rpy="0 0 0"/>
-    </joint>
-    <gazebo reference="imu_link">
-    <gravity>false</gravity>
-    <sensor name="imu_sensor" type="imu">
-      <always_on>true</always_on>
-      <update_rate>100</update_rate>
-      <visualize>true</visualize>
-      <topic>__default_topic__</topic>
-      <plugin filename="libgazebo_ros_imu_sensor.so" name="imu_plugin">
-        <topicName>imu</topicName>
-        <bodyName>imu_link</bodyName>
-        <updateRateHZ>10.0</updateRateHZ>
-        <gaussianNoise>0.0</gaussianNoise>
-        <xyzOffset>0 0 0</xyzOffset>
-        <rpyOffset>0 0 0</rpyOffset>
-        <frameName>imu_link</frameName>
-        <initialOrientationAsReference>false</initialOrientationAsReference>
-      </plugin>
-      <pose>0 0 0 0 0 0</pose>
-    </sensor>
-  </gazebo>
 </robot>
