Commit message: HeadModule

File: real/description/example_robot.urdf.xacro (robot description, xacro)
@@ -2,8 +2,7 @@
 <robot xmlns:xacro="http://www.ros.org/wiki/xacro"  name="INSECTOIDv1">
     <xacro:include filename="patterns.xacro"/>
-    <xacro:include filename="IMUsim.xacro"/>
-    <xacro:include filename="example_gazebo.xacro" />
-    <xacro:include filename="ros2_control.xacro"/>
-    <xacro:include filename="lidar.xacro"/>
+    <!--<xacro:include filename="example_gazebo.xacro" />-->
+    <!--<xacro:include filename="ros2_control.xacro"/>-->
+    <!--<xacro:include filename="lidar.xacro"/>-->
     <!---->
 	<link name="base_link"></link>

File: real/description/patterns.xacro (robot description, xacro)
@@ -2,9 +2,11 @@
 <robot xmlns:xacro="http://www.ros.org/wiki/xacro">
 <!--Models-->
-    <xacro:property name="base_path" value="file:////home/zega/Desktop/ros_dev/src/my_gazebo/meshes/base1.dae" />
-    <xacro:property name="arm_path_1" value="file:////home/zega/Desktop/ros_dev/src/my_gazebo/meshes/l-1.dae" />
-    <xacro:property name="arm_path_2" value="file:////home/zega/Desktop/ros_dev/src/my_gazebo/meshes/l-2.dae" />
-    <xacro:property name="arm_path_3" value="file:////home/zega/Desktop/ros_dev/src/my_gazebo/meshes/l-3.dae" />
-    <xacro:property name="camera" value="file:////home/zega/Desktop/ros_dev/src/my_gazebo/meshes/kinect.dae" />
+    <xacro:property name="package_root" value="file://$(find real)" />
+    <xacro:property name="meshes_dir" value="${package_root}/meshes" />
+    <xacro:property name="base_path" value="${meshes_dir}/base1.dae" />
+    <xacro:property name="arm_path_1" value="${meshes_dir}/l-1.dae" />
+    <xacro:property name="arm_path_2" value="${meshes_dir}/l-2.dae" />
+    <xacro:property name="arm_path_3" value="${meshes_dir}/l-3.dae" />
+    <xacro:property name="camera" value="${meshes_dir}/kinect.dae" />
  <!--Models-->
     <material name="white">
@@ -44,5 +46,5 @@
 <!--LEG MACROS-->
     <xacro:macro name="leg_section_joint" params="joint_name joint_axis joint_xyz joint_parent joint_child lower_limit upper_limit ">
-		<joint name="${joint_name}" type="revolute">
+		<joint name="${joint_name}" type="fixed">
 		    <origin xyz="${joint_xyz}" />
 		    <parent link="${joint_parent}" />
